File: hardware1551/bss138.kicad_sch (KiCad schematic)
At the start: 3 parts, among them Q2 BSS138

Commit message: 1551 version with Fake6523_hw_checked by ZXByteman
Parts:
- renumbered Q2 to Q1, R5 to R3, R6 to R4

Commit message: updates and cleanups
Parts:
- removed R3, R4: 10k, Resistor_SMD:R_0603_1608Metric, symbol Device:R
- added R1, R2: 10k, Resistor_SMD:R_0805_2012Metric_Pad1.20x1.40mm_HandSolder, symbol Device:R
Connections:
- net +5V: now also R2.1
- net HIGH: now also R2.2
- net LOW: now also R1.2
- net +3.3V renamed +3V3
- net +3V3: now also R1.1
