File: hardware1551/bss138.kicad_sch (KiCad schematic)
At the start: 3 parts, among them Q1 BSS138

Commit message: board for 1551 with correct dimensions and spacing between CPU and TPI, routed
Parts:
- Q1: JLCPCB Part # (none) -> C78284; JLCPCB URL (none) -> https://jlcpcb.com/partdetail/79418-BSS138/C78284; MFR.Part # (none) -> BSS138
Changed lines of the file:
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@@
+			)
+		)
+		(property "JLCPCB Part #" "C78284"
+			(at 146.05 86.36 90)
+			(effects
+				(font
+					(size 1.27 1.27)
+				)
+				(hide yes)
+			)
+		)
+		(property "JLCPCB URL" "https://jlcpcb.com/partdetail/79418-BSS138/C78284"
+			(at 146.05 86.36 90)
+			(effects
+				(font
+					(size 1.27 1.27)
+				)
+				(hide yes)
+			)
+		)
+		(property "MFR.Part #" "BSS138"
+			(at 146.05 86.36 90)
+			(effects
+				(font
+					(size 1.27 1.27)
+				)
+				(hide yes)
 			)
 		)
@@
 				(path "/7c37ffbe-d8d1-4c30-ad42-fd3ef959e14d/75d2c140-5eb5-44c3-a43e-847105354624"
 					(reference "Q2")
+					(unit 1)
+				)
+				(path "/7c37ffbe-d8d1-4c30-ad42-fd3ef959e14d/93c5a10e-e0aa-481a-bb6b-5a0241e2376b"
+					(reference "Q4")
 					(unit 1)
 				)
@@
 				(path "/7c37ffbe-d8d1-4c30-ad42-fd3ef959e14d/75d2c140-5eb5-44c3-a43e-847105354624"
 					(reference "#PWR010")
+					(unit 1)
+				)
+				(path "/7c37ffbe-d8d1-4c30-ad42-fd3ef959e14d/93c5a10e-e0aa-481a-bb6b-5a0241e2376b"
+					(reference "#PWR0106")
 					(unit 1)
 				)
@@
 					(unit 1)
 				)
+				(path "/7c37ffbe-d8d1-4c30-ad42-fd3ef959e14d/93c5a10e-e0aa-481a-bb6b-5a0241e2376b"
+					(reference "R9")
+					(unit 1)
+				)
 			)
 		)
@@
 					(unit 1)
 				)
+				(path "/7c37ffbe-d8d1-4c30-ad42-fd3ef959e14d/93c5a10e-e0aa-481a-bb6b-5a0241e2376b"
+					(reference "#PWR0105")
+					(unit 1)
+				)
 			)
 		)
@@
 					(unit 1)
 				)
+				(path "/7c37ffbe-d8d1-4c30-ad42-fd3ef959e14d/93c5a10e-e0aa-481a-bb6b-5a0241e2376b"
+					(reference "R10")
+					(unit 1)
+				)
