File: hardware1551/1551-rePico.kicad_sch (KiCad schematic)
At the start: 14 parts, among them J1 Display Connector, J2 Display Power, J3 Conn_01x05_Pin, J4 SD Card Module Connector, J5 Conn_01x01_Pin, J6 EXT_5V, J7 RESET_1541, SW1 RESET, U1 Pico

Commit message: 1551 version with Fake6523_hw_checked by ZXByteman
Parts:
- removed J1: Display Connector, Connector_PinSocket_2.54mm:PinSocket_2x02_P2.54mm_Vertical, symbol Connector_Generic:Conn_02x02_Odd_Even
- removed J2: Display Power, Connector_PinHeader_2.54mm:PinHeader_1x03_P2.54mm_Vertical, symbol Connector_Generic:Conn_01x03
- removed J3: Conn_01x05_Pin, Connector_PinHeader_2.54mm:PinHeader_1x05_P2.54mm_Vertical, symbol Connector:Conn_01x05_Pin
- removed J4: SD Card Module Connector, Connector_PinSocket_2.54mm:PinSocket_2x08_P2.54mm_Vertical, symbol Connector_Generic:Conn_02x08_Odd_Even
- removed J6: EXT_5V, Connector_PinHeader_2.54mm:PinHeader_1x02_P2.54mm_Vertical, symbol Connector_Generic:Conn_01x02
- removed J7: RESET_1541, Connector_PinHeader_2.54mm:PinHeader_1x02_P2.54mm_Vertical, symbol Connector_Generic:Conn_01x02
- removed R3: 10k, Resistor_THT:R_Axial_DIN0207_L6.3mm_D2.5mm_P10.16mm_Horizontal, symbol Device:R
- removed SW1: RESET, Button_Switch_THT:SW_PUSH_6mm_H5mm, symbol Switch:SW_Push
- added C2, C3, C4, C5: 0.1uF, Capacitor_SMD:C_0805_2012Metric_Pad1.18x1.45mm_HandSolder, symbol Device:C_Small
- added J1: 0.96_I2C_OLED, Connector_PinHeader_2.54mm:PinHeader_1x04_P2.54mm_Vertical, symbol Connector_Generic:Conn_01x04
- added J10: TCBM, Connector_IDC:IDC-Header_2x08_P2.54mm_Vertical, symbol Connector_Generic:Conn_02x08_Odd_Even
- added J11: JTAG, Connector_PinHeader_2.54mm:PinHeader_1x06_P2.54mm_Vertical, symbol Connector_Generic:Conn_01x06
- added J6: Conn_01x05, Connector_PinHeader_2.54mm:PinHeader_1x05_P2.54mm_Vertical, symbol Connector_Generic:Conn_01x05
- added J8: SD CARD, Connector_PinHeader_2.54mm:PinHeader_1x06_P2.54mm_Vertical, symbol Connector_Generic:Conn_01x06
- added JP3, JP4: SolderJumper_3_Bridged12, Jumper:SolderJumper-3_P1.3mm_Bridged12_RoundedPad1.0x1.5mm_NumberLabels, symbol Jumper:SolderJumper_3_Bridged12
- added U3: XC9572XL-VQ64, Package_QFP:TQFP-64_10x10mm_P0.5mm, symbol CPLD_Xilinx:XC9572XL-VQ64
- added U4: 6523 (pins), Package_DIP:DIP-40_W15.24mm, symbol 65xx:6523
- added U5: 6510T (pins), Package_DIP:DIP-40_W15.24mm, symbol 65xx:6510T
- added U6: 6510T (socket for chip), Package_DIP:DIP-40_W15.24mm, symbol 65xx:6510T
Connections:
- net +3.3V: no longer R1.1, R2.1
- net +5V: now also U4.20 (VDD), U5.5 (VCC), U6.5 (VCC)
- net GND: now also U1.33 (AGND), C2.2, C3.2, C4.2, C5.2, J10.1 (Pin_1), J10.16 (Pin_16), J11.6 (Pin_6), J6.5 (Pin_5), J8.6 (Pin_6), JP3.1 (A), JP4.3 (B), U3.14 (GND), U3.21 (GND), U3.41 (GND), U3.54 (GND), U4.1 (VSS), U5.20 (VSS), U6.20 (VSS)
- net I2C_SCL: now also R2.2, J1.3 (Pin_3); no longer R1.2
- net I2C_SDA: now also R1.2, J1.4 (Pin_4); no longer R2.2
- net ~{RESET_3V3}: now reaches U1.30 (RUN)
- net ~{RESET_3V3}: now also U3.51 (P51)
- net ROT_CLK: now reaches U1.31 (GPIO26_ADC0)
- net ROT_CLK: now also J6.1 (Pin_1)
- net ROT_DT: now reaches U1.32 (GPIO27_ADC1)
- net ROT_DT: now also J6.2 (Pin_2)
- net ROT_SW: now reaches U1.34 (GPIO28_ADC2)
- net ROT_SW: now also J6.3 (Pin_3)
- net CS renamed SD_CS
- net SD_CS: now also J8.2 (Pin_2)
- net MISO renamed SD_MISO
- net SD_MISO: now also J8.5 (Pin_5)
- net MOSI renamed SD_MOSI
- net SD_MOSI: now also J8.3 (Pin_3)
- net SCK renamed SD_SCK
- net SD_SCK: now also J8.4 (Pin_4)
- net _BRDY renamed BYTE_READY_3V3
- net BYTE_READY_3V3: now also U3.19 (P19)
- net _MTR renamed MTR_3V3
- net _OE renamed MODE_3V3
- net MODE_3V3: now also U3.50 (P50)
- net _PA0 renamed YB0
- net YB0: now also U3.22 (P22)
- net _PA1 renamed YB1
- net YB1: now also U3.27 (P27)
- net _PA2 renamed YB2
- net YB2: now also U3.32 (P32)
- net _PA3 renamed YB3
- net YB3: now also U3.33 (P33)
- net _PA4 renamed YB4
- net YB4: now also U3.34 (P34)
- net _PA5 renamed YB5
- net YB5: now also U3.35 (P35)
- net _PA6 renamed YB6
- net YB6: now also U3.36 (P36)
- net _PA7 renamed YB7
- net YB7: now also U3.38 (P38)
- net _SOE renamed SOE_3V3
- net SOE_3V3: now also U3.18 (P18)
- net _SOE_GA renamed DEVNUM_3V3
- net DEVNUM_3V3: now also U3.52 (P52)
- net _STP0 renamed STP0_3V3
- net _STP1 renamed STP1_3V3
- net _SYNC renamed SYNC_3V3
- net SYNC_3V3: now also U3.56 (P56)
- new net: J1.1 (Pin_1), JP3.2 (C)
- new net: J1.2 (Pin_2), JP4.2 (C)
- new net +3V3: C2.1, C3.1, C4.1, C5.1, J11.1 (Pin_1), J6.4 (Pin_4), J8.1 (Pin_1), JP3.3 (B), JP4.1 (A), R1.1, R2.1, U3.26 (VCCIO), U3.3 (VCC), U3.37 (VCC), U3.55 (VCCIO)
- new net A0: U3.45 (P45), U4.24 (RS0), U5.6 (A0), U6.6 (A0)
- new net A1: U3.44 (P44), U4.23 (RS1), U5.7 (A1), U6.7 (A1)
- new net A10: U5.16 (A10), U6.16 (A10)
- new net A11: U5.17 (A11), U6.17 (A11)
- new net A12: U5.18 (A12), U6.18 (A12)
- new net A13: U5.19 (A13), U6.19 (A13)
- new net A14: U5.21 (A14), U6.21 (A14)
- new net A15: U5.22 (A15), U6.22 (A15)
- new net A2: U3.43 (P43), U4.22 (RS2), U5.8 (A2), U6.8 (A2)
- new net A3: U5.9 (A3), U6.9 (A3)
- new net A4: U5.10 (A4), U6.10 (A4)
- new net A5: U5.11 (A5), U6.11 (A5)
- new net A6: U5.12 (A6), U6.12 (A6)
- new net A7: U5.13 (A7), U6.13 (A7)
- new net A8: U5.14 (A8), U6.14 (A8)
- new net A9: U5.15 (A9), U6.15 (A9)
- new net ACK: J10.13 (Pin_13), U3.57 (P57), U4.32 (PC7)
- new net ACT: U5.27 (P3), U6.27 (P3)
- new net AEC: U5.4 (AEC), U6.4 (AEC)
- new net BYTE_LATCHED: U3.20 (P20), U5.23 (P7), U6.23 (P7)
- new net D0: U3.60 (P60), U4.33 (D0), U5.38 (D0), U6.38 (D0)
- new net D1: U3.1 (P1), U4.34 (D1), U5.37 (D1), U6.37 (D1)
- new net D2: U3.2 (I/O/GTS2), U4.35 (D2), U5.36 (D2), U6.36 (D2)
- new net D3: U3.4 (P4), U4.36 (D3), U5.35 (D3), U6.35 (D3)
- new net D4: U3.5 (I/O/GTS1), U4.37 (D4), U5.34 (D4), U6.34 (D4)
- new net D5: U3.6 (P6), U4.38 (D5), U5.33 (D5), U6.33 (D5)
- new net D6: U3.7 (P7), U4.39 (D6), U5.32 (D6), U6.32 (D6)
- new net D7: U3.63 (P63), U4.40 (D7), U5.31 (D7), U6.31 (D7)
- new net DAV: J10.11 (Pin_11), U3.49 (P49), U4.28 (PC3)
- new net DEV: J10.2 (Pin_2), U3.48 (P48), U4.27 (PC2)
- new net DEVNUM_BRD: U4.30 (PC5)
- new net DIO1: J10.3 (Pin_3), U3.9 (P9), U4.2 (PA0)
- new net DIO2: J10.4 (Pin_4), U3.10 (P10), U4.3 (PA1)
- new net DIO3: J10.5 (Pin_5), U3.11 (P11), U4.4 (PA2)
- new net DIO4: J10.6 (Pin_6), U3.12 (P12), U4.5 (PA3)
- new net DIO5: J10.7 (Pin_7), U3.13 (P13), U4.6 (PA4)
- new net DIO6: J10.8 (Pin_8), U3.15 (I/O/GCK1), U4.7 (PA5)
- new net DIO7: J10.9 (Pin_9), U3.16 (I/O/GCK2), U4.8 (PA6)
- new net DIO8: J10.10 (Pin_10), U3.17 (I/O/GCK3), U4.9 (PA7)
- new net DS0: U5.25 (P5), U6.25 (P5)
- new net DS1: U5.24 (P6), U6.24 (P6)
- new net MODE: U4.29 (PC4)
- new net MTR: U5.28 (P2), U6.28 (P2)
- new net PHI0: U3.31 (P31), U5.2 (ϕ0), U6.2 (ϕ0)
- new net PHI2: U3.25 (P25), U5.40 (ϕ2), U6.40 (ϕ2)
- new net R/~{W}: U3.24 (P24), U5.39 (R/~{W}), U6.39 (R/~{W})
- new net STATUS0: J10.12 (Pin_12), U3.46 (P46), U4.25 (PC0)
- new net STATUS1: J10.14 (Pin_14), U3.47 (P47), U4.26 (PC1)
- new net STP0: U5.29 (P1), U6.29 (P1)
- new net STP1: U5.30 (P0), U6.30 (P0)
- new net SYNC: U4.31 (PC6)
- new net TCK: J11.3 (Pin_3), U3.30 (TCK)
- new net TDI: J11.4 (Pin_4), U3.28 (TDI)
- new net TDO: J11.5 (Pin_5), U3.53 (TDO)
- new net TMS: J11.2 (Pin_2), U3.29 (TMS)
- new net WPS: U5.26 (P4), U6.26 (P4)
- new net XR/~{W}: U3.40 (P40), U4.19 (R/~{W})
- new net YB0_BRD: U4.10 (PB0)
- new net YB1_BRD: U4.11 (PB1)
- new net YB2_BRD: U4.12 (PB2)
- new net YB3_BRD: U4.13 (PB3)
- new net YB4_BRD: U4.14 (PB4)
- new net YB5_BRD: U4.15 (PB5)
- new net YB6_BRD: U4.16 (PB6)
- new net YB7_BRD: U4.17 (PB7)
- new net ~{CS_TPI}: U3.39 (P39), U4.18 (~{CS})
- new net ~{IRQ}: U5.3 (~{IRQ}), U6.3 (~{IRQ})
- new net ~{RESET}: J10.15 (Pin_15), U3.64 (I/O/GSR), U4.21 (~{RST}), U5.1 (~{RES}), U6.1 (~{RES})
- no-connect marks 4 -> 9
Other:
- removed sheet VIA 6522 Sockel
- added sheet BSS138_6 (bss138.kicad_sch)
- added sheet BSS138_7 (bss138.kicad_sch)
- added sheet BSS138_8 (bss138.kicad_sch)
- note added: "23x18mm SD Card module 3.3v"
- note added: "NOTE: ACK/DAV naming reversed to keep the TCBM2SD connector intact NOTE: ACK here is controller's ACK output and goes to cable pin 13 (drive's DAV input) NOTE: DAV here is controller's DAV input and goes to cable pin 11 (drive's ACK output) NOTE: DEVNUM_BRD is shorted to GND onboard with hard to use J1 to be cut to pull it up control it on daughterboard NOTE: ~{CS_TPI} is the signal we need to cl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"
- note added: "NOTE: DEVNUM_3V3 - driven by Pico to choose device number, NOT connected to DEVNUM_BRD"
- note added: "NOTE: WPS can be disconnected from board and controled on daughterboard NOTE: DS0/DS1 not connected to pico, no way for unusual formats like SuperDOS? (unless it's not needed at all for G64) NOTE: Phi2 NC onboard, AEC pulled up"
- note added: "NOTE: no macrocells left to use CPLD for level shifting NOTE: all _3V3 signals are for Pico only, NOT for board NOTE: YB0..7 are for Pico only TODO: RESET_3V3, MODE_3V3, SYNC_3V3 NOTE: XR/~{W} comes from GATE ARRAY, it is NOT CPU's R/~{W} CPLD firmware can be later changed to use R/~{W} + Phi0/Phi2 without gate array"
- note added: "Rotary encoder (KY-040)"
- note added: "Switch BOTH JP3/JP4 for VCC/GND/SCL/SDA or GND/VCC/SCL/SDA"
- note added: "TODO: Pico decides about device number - output on GPIO3 0 or 1"
- note added: "WPS"
- note added: "WPS: to U8-pin 1 (74LS14), R18, connector P5-12"
- note added: "no need to level shift these if they ONLY go to CPLD NOTE: YBx=PBx goes ONLY to CPLD can be disconnected from the board NOTE: same with MODE, SYNC from port C - but be sure about existing pullups/pulldowns"
- note removed: "Externe Spannungsversorgung, nur verwenden wenn _kein_ Floppy-Netzteil angeschlossen wird !"
- note removed: "Jumper Normal offen"
- note removed: "Pinbelegung für DrehDrückGeber PIN1: GND PIN2: + PIN3: SW PIN4: DT PIN5: CLK"
- title: 1541-rePico -> 1551-rePico
- moved on the sheet: R1, R2

Commit message: updates and cleanups
Parts:
- removed C1: 47µF, Capacitor_THT:CP_Radial_D5.0mm_P2.50mm, symbol Device:CP
- removed R1, R2: 1.8k, Resistor_SMD:R_0805_2012Metric, symbol Device:R
- added C1: 47µF, Capacitor_THT:CP_Radial_D5.0mm_P2.50mm, symbol Device:C_Polarized
- added JP1: ~, Jumper:SolderJumper-2_P1.3mm_Open_RoundedPad1.0x1.5mm, symbol Jumper:SolderJumper_2_Open
Connections:
- net +3.3V is gone; now on net +3V3: U1.36 (3V3)
- net +5V: now also C1.1
- net GND: now also C1.2
- net ~{RESET_3V3}: now also JP1.1 (A); no longer U1.30 (RUN)
- new net: JP1.2 (B), U1.30 (RUN)
- no-connect marks 9 -> 10
Other:
- company: (none) -> YTM Enterprises

Commit message: drop SOE, add pullups, drive WPS directly to CPU pin (open drain)
Parts:
- removed J5: Conn_01x01_Pin, Connector_PinHeader_2.00mm:PinHeader_1x01_P2.00mm_Vertical, symbol Connector:Conn_01x01_Pin
- added R11, R12, R13, R14, R7, R8: 10k, Resistor_SMD:R_0805_2012Metric_Pad1.20x1.40mm_HandSolder, symbol Device:R
Connections:
- net +3V3: now also R11.1, R12.1, R13.1, R14.1, R7.1, R8.1
- net BYTE_READY_3V3: now also R8.2
- net I2C_SCL: now also R13.2
- net I2C_SDA: now also R14.2
- net MODE_3V3: now also R11.2
- net SYNC_3V3: now also R12.2
- net ~{RESET_3V3}: now also R7.2
- net WPS_3V3: now reaches U1.7 (GPIO5)
- net SOE_3V3: no longer names the net of U3.18 (P18)
- net SOE_3V3: no longer U1.1 (GPIO0)
- no-connect marks 10 -> 23
Other:
- added sheet BSS138_9 (bss138.kicad_sch)
- note added: "Pico firmware TODO: - GPIO0: SOE not used (always high), can be fixed in firmware to true - GPIO3: Pico decides about device number - 0 or 1 - GPIO5: switch driver from high/low to hi-z/low"
- note removed: "TODO: Pico decides about device number - output on GPIO3 0 or 1"
- note removed: "WPS"
- note removed: "WPS: to U8-pin 1 (74LS14), R18, connector P5-12"
