File: hardware1551/1551-rePico.kicad_sch (KiCad schematic)
At the start: 29 parts, among them J1 0.96_I2C_OLED, J10 TCBM, J11 JTAG, J6 Conn_01x05, J8 SD CARD, U1 Pico, U3 XC9572XL-VQ64, U4 6523 (pins), U5 6510T (pins), U6 6510T (socket for chip)

Commit message: confirm how LED works (ACT=0 is ON)
Other:
- note added: "P4: WPS, but don't connect it to mainboard b/c it's an output of U8 inverter, with no other mechanism to drive it low P7: BYTE_LATCHED, not connected either (gate array could drive it) P3: ACT led goes between pins 8 (+5V) and 9 (ACT) of P5 (pin 1 is GND) (on 1551 separated from LED with buffer)"
- note added: "Pico firmware: - GPIO0: SOE not used (always high), set in firmware to always true OR can be used to test 2MHz clock (PHI0) for 6502 - GPIO3: Pico decides about device number - 0 or 1 OR drives ~{IRQ} for 6502"
- note removed: "Pico firmware TODO: - GPIO0: SOE not used (always high), can be fixed in firmware to true OR can be used to test 2MHz clock (PHI0) for 6502 - GPIO3: Pico decides about device number - 0 or 1 OR can be used to test 100Hz (IRQ) for 6502 - GPIO5: switch driver from high/low to hi-z/low"
- note removed: "WPS would be on P4, but don't connect it to mainboard b/c it's an output of U8 inverter, with no mechanism it drives it low BYTE_LATCHED would be on P7, not connected either (gate array ould drive it)"
Changed lines of the file:
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@@
 		)
 	)
-	(text "WPS would be on P4, but don't connect it to mainboard\nb/c it's an output of U8 inverter, with no mechanism\nit drives it low\nBYTE_LATCHED would be on P7, not connected either\n(gate array ould drive it)"
+	(text "P4: WPS, but don't connect it to mainboard\n    b/c it's an output of U8 inverter, with no\n    other mechanism to drive it low\nP7: BYTE_LATCHED, not connected either\n    (gate array could drive it)\nP3: ACT led goes between pins 8 (+5V) and 9 (ACT) of P5 (pin 1 is GND)\n    (on 1551 separated from LED with buffer)"
 		(exclude_from_sim no)
 		(at 355.092 192.024 0)
@@
 		)
 	)
-	(text "Pico firmware TODO:\n- GPIO0: SOE not used (always high), can be fixed in firmware to true\n  OR can be used to test 2MHz clock (PHI0) for 6502\n- GPIO3: Pico decides about device number - 0 or 1\n  OR can be used to test 100Hz (IRQ) for 6502\n- GPIO5: switch driver from high/low to hi-z/low"
+	(text "Pico firmware:\n- GPIO0: SOE not used (always high), set in firmware to always true\n  OR can be used to test 2MHz clock (PHI0) for 6502\n- GPIO3: Pico decides about device number - 0 or 1\n  OR drives ~{IRQ} for 6502"
 		(exclude_from_sim no)
 		(at 200.66 69.596 0)
