File: hardware-1551-III-Pico/1551-III-Pico.kicad_sch (KiCad schematic)
At the start: 43 parts, among them J1 DC IN, J3 TCBM, J4 Mini-DIN-7, J8 Module_Panel, M1 Mounting, M2 Mounting, M3 Mounting, M4 Mounting, Q1 MMBT3904, Q2 MMBT3904, Q3 MMBT3904, Q4 MMBT3904

Commit message: 1551 board that might actually work
Parts:
- removed A1: Raspberry PI 3A/3B, RPI:Raspberry_Pi_3B_Socketed_THT_FaceDown_MountingHoles, symbol raspberry_pi:Raspberry_Pi_2_3
- removed BZ1: Buzzer, small_buzzer:Buzzer_12x9.5RM7.6, symbol Device:Speaker
- removed J4: Mini-DIN-7, Conn_DIN_round:Mini_DIN_round_7_canned, symbol Connector:Mini-DIN-7
- removed JP1, JP2: SolderJumper_3_Bridged12, Jumper:SolderJumper-3_P1.3mm_Bridged12_RoundedPad1.0x1.5mm_NumberLabels, symbol Jumper:SolderJumper_3_Bridged12
- removed Q2, Q3, Q4: MMBT3904, Package_TO_SOT_SMD:SOT-23_Handsoldering, symbol Transistor_BJT:MMBT3904
- removed R10, R11, R4, R5, R6, R7, R9: 3.3K, Resistor_SMD:R_0805_2012Metric_Pad1.20x1.40mm_HandSolder, symbol Device:R
- added C10, C11, C12, C13, C2, C3, C4, C5, C6, C8: 0.1uF, Capacitor_SMD:C_0805_2012Metric_Pad1.18x1.45mm_HandSolder, symbol Device:C_Small
- added C7: 10nF, symbol Device:C_Small
- added C9: 100nF, symbol Device:C_Small
- added J2: SD CARD, Connector_PinHeader_2.54mm:PinHeader_1x06_P2.54mm_Vertical, symbol Connector_Generic:Conn_01x06
- added J5: JTAG, Connector_PinHeader_2.54mm:PinHeader_1x06_P2.54mm_Vertical, symbol Connector_Generic:Conn_01x06
- added J6: Conn_01x02_Pin, Connector_PinHeader_2.54mm:PinHeader_1x02_P2.54mm_Vertical, symbol Connector:Conn_01x02_Pin
- added JP1: ~, Jumper:SolderJumper-2_P1.3mm_Open_RoundedPad1.0x1.5mm, symbol Jumper:SolderJumper_2_Open
- added JP2, JP3: Jumper_2_Bridged, Connector_PinHeader_2.54mm:PinHeader_1x02_P2.54mm_Vertical, symbol Jumper:Jumper_2_Bridged
- added R1, R16, R2, R22, R25, R3: 3.3K, Resistor_SMD:R_0805_2012Metric_Pad1.20x1.40mm_HandSolder, symbol Device:R
- added R23: 100, Resistor_SMD:R_0805_2012Metric_Pad1.20x1.40mm_HandSolder, symbol Device:R
- added R24: 150K, Resistor_SMD:R_0805_2012Metric_Pad1.20x1.40mm_HandSolder, symbol Device:R
- added R26: 68, Resistor_SMD:R_0805_2012Metric_Pad1.20x1.40mm_HandSolder, symbol Device:R
- added SWDBG1: DEBUG, Connector_PinHeader_2.54mm:PinHeader_1x03_P2.54mm_Vertical, symbol Connector_Generic:Conn_01x03
- added U1: Pico, RPi_Pico:RPi_Pico_SMD_TH, symbol MCU_RaspberryPi_and_Boards:Pico
- added U2: 6510T, Package_DIP:DIP-40_W15.24mm, symbol 65xx:6510T
- added U3: XC9572XL-VQ64, Package_QFP:TQFP-64_10x10mm_P0.5mm, symbol CPLD_Xilinx:XC9572XL-VQ64
- added U4: 27C512, Package_DIP:DIP-28_W15.24mm_Socket_LongPads, symbol Memory_EPROM:27C512
- added U5: 74LS139, Package_DIP:DIP-16_W7.62mm_Socket_LongPads, symbol 74xx:74LS139
- added U6: 74LS00, Package_DIP:DIP-14_W7.62mm_Socket_LongPads, symbol 74xx:74LS00
- added U7: KM62256CLP, Package_DIP:DIP-28_W15.24mm_Socket_LongPads, symbol Memory_RAM:KM62256CLP
- added U8: NE555P, Package_DIP:DIP-8_W7.62mm, symbol Timer:NE555P
- added U9: 74AHCT1G125, symbol 74xGxx:74AHCT1G125
- added Y1: 2MHz, Oscillator:Oscillator_DIP-14, symbol Oscillator:CXO_DIP14
- renumbered C6 to C1, D2 to D1, J8 to J4, R17 to R10, R1 to R11, R2 to R12, R3 to R13, R18 to R14, R19 to R15, R20 to R17, R21 to R18, R22 to R19, R23 to R20, R24 to R21, R12 to R4, R13 to R5, R14 to R6, R15 to R7, R16 to R9
Connections:
- net RPI_LED is gone; now on net ACT_3V3: R13.1
- net +3.3V: now also R16.1
- net +5V: now also C10.1, C11.1, C12.1, C13.1, C6.1, C8.1, R22.1, R24.1, R25.1, U1.39 (VSYS), U2.5 (VCC), U4.28 (VCC), U5.16 (VCC), U6.14 (VCC), U7.28 (VCC), U8.4 (~{RST}), U8.8 (VCC), U9.5 (VCC), Y1.14 (Vcc)
- net ACK: now also U3.57 (P57)
- net DAV: now also U3.49 (P49)
- net DEV: now also U3.48 (P48)
- net DIO1: now also U3.9 (P9)
- net DIO2: now also U3.10 (P10)
- net DIO3: now also U3.11 (P11)
- net DIO4: now also U3.12 (P12)
- net DIO5: now also U3.13 (P13)
- net DIO6: now also U3.15 (I/O/GCK1)
- net DIO7: now also U3.16 (I/O/GCK2)
- net DIO8: now also U3.17 (I/O/GCK3)
- net GND: now also C10.2, C11.2, C12.2, C13.2, C2.2, C3.2, C4.2, C5.2, C6.2, C7.2, C8.2, C9.2, J2.6 (Pin_6), J5.6 (Pin_6), J6.2 (Pin_2), U1.13 (GND), U1.18 (GND), U1.23 (GND), U1.28 (GND), U1.3 (GND), U1.33 (AGND), U1.38 (GND), U1.8 (GND), U2.20 (VSS), U3.14 (GND), U3.21 (GND), U3.41 (GND), U3.54 (GND), U4.14 (GND), U5.1 (E), U5.14 (A0), U5.8 (GND), U6.7 (GND), U7.14 (GND), U8.1 (GND), U9.1, U9.3 (GND), Y1.7 (GND)
- net I2C_SCL: now also U1.27 (GPIO21)
- net I2C_SDA: now also U1.26 (GPIO20)
- net STATUS0: now also U3.46 (P46)
- net STATUS1: now also U3.47 (P47)
- net ~{RESET_3V3}: now also JP1.1 (A), U3.51 (P51)
- net ~{RESET}: now also U2.1 (~{RES}), U3.64 (I/O/GSR)
- net ACT_3V3: now reaches Q1.3 (C)
- net ACT_3V3: now also R16.2
- net at Q1.1 (B): now also R8.1
- net CAS_WRITE renamed ACT
- net ACT: now also U2.27 (P3)
- net SW1_ENTER renamed ROT_SW
- net ROT_SW: now also U1.34 (GPIO28_ADC2)
- net SW2_UP renamed ROT_CLK
- net ROT_CLK: now also U1.31 (GPIO26_ADC0)
- net SW3_DOWN renamed ROT_DT
- net ROT_DT: now also U1.32 (GPIO27_ADC1)
- new net: C7.1, U8.5 (CONT)
- new net: JP2.2 (B), Y1.8 (OUT)
- new net: U6.12, U6.13, U6.8
- new net: R26.2, U9.4
- new net: J6.1 (Pin_1), R22.2, U4.1 (A15)
- new net: R23.1, R24.2, U8.7 (DISCH)
- new net: JP3.2 (B), U8.3 (OUT)
- new net: C9.1, R23.2, U8.2 (TRIG), U8.6 (THRES)
- new net: SWDBG1.1 (Pin_1), U1.41 (SWCLK)
- new net: SWDBG1.2 (Pin_2), U1.42 (GND)
- new net: SWDBG1.3 (Pin_3), U1.43 (SWDIO)
- new net: U6.3, U6.4, U6.5
- new net: JP1.2 (B), U1.30 (RUN)
- new net +3V3: C2.1, C3.1, C4.1, C5.1, J2.1 (Pin_1), J5.1 (Pin_1), R1.1, R2.1, R3.1, U1.36 (3V3), U3.26 (VCCIO), U3.3 (VCC), U3.37 (VCC), U3.55 (VCCIO)
- new net A0: U2.6 (A0), U3.45 (P45), U4.10 (A0), U7.10 (A0)
- new net A1: U2.7 (A1), U3.44 (P44), U4.9 (A1), U7.9 (A1)
- new net A10: U2.16 (A10), U4.21 (A10), U7.21 (A10)
- new net A11: U2.17 (A11), U4.23 (A11), U7.23 (A11)
- new net A12: U2.18 (A12), U4.2 (A12), U7.2 (A12)
- new net A13: U2.19 (A13), U4.26 (A13), U5.13 (A1), U7.26 (A13)
- new net A14: U2.21 (A14), U4.27 (A14), U5.3 (A1)
- new net A15: U2.22 (A15), U5.2 (A0), U7.1 (A14)
- new net A2: U2.8 (A2), U3.43 (P43), U4.8 (A2), U7.8 (A2)
- new net A3: U2.9 (A3), U4.7 (A3), U7.7 (A3)
- new net A4: U2.10 (A4), U4.6 (A4), U7.6 (A4)
- new net A5: U2.11 (A5), U4.5 (A5), U7.5 (A5)
- new net A6: U2.12 (A6), U4.4 (A6), U7.4 (A6)
- new net A7: U2.13 (A7), U4.3 (A7), U7.3 (A7)
- new net A8: U2.14 (A8), U4.25 (A8), U7.25 (A8)
- new net A9: U2.15 (A9), U4.24 (A9), U7.24 (A9)
- new net AEC: U2.4 (AEC)
- new net BYTE_LATCHED: U2.23 (P7), U3.20 (P20)
- new net BYTE_READY_3V3: R1.2, U1.29 (GPIO22), U3.19 (P19)
- new net D0: U2.38 (D0), U3.60 (P60), U4.11 (D0), U7.11 (Q0)
- new net D1: U2.37 (D1), U3.1 (P1), U4.12 (D1), U7.12 (Q1)
- new net D2: U2.36 (D2), U3.2 (I/O/GTS2), U4.13 (D2), U7.13 (Q2)
- new net D3: U2.35 (D3), U3.4 (P4), U4.15 (D3), U7.15 (Q3)
- new net D4: U2.34 (D4), U3.5 (I/O/GTS1), U4.16 (D4), U7.16 (Q4)
- new net D5: U2.33 (D5), U3.6 (P6), U4.17 (D5), U7.17 (Q5)
- new net D6: U2.32 (D6), U3.7 (P7), U4.18 (D6), U7.18 (Q6)
- new net D7: U2.31 (D7), U3.63 (P63), U4.19 (D7), U7.19 (Q7)
- new net DEVNUM_3V3: U1.5 (GPIO3), U3.52 (P52)
- new net DS0: U2.25 (P5)
- new net DS1: U2.24 (P6)
- new net MODE_3V3: R2.2, U1.2 (GPIO1), U3.50 (P50)
- new net MTR: U2.28 (P2)
- new net MTR_3V3: U1.6 (GPIO4)
- new net PHI0: JP2.1 (A), U2.2 (ϕ0), U3.31 (P31)
- new net PHI2: U2.40 (ϕ2), U3.25 (P25)
- new net R/~{W}: U2.39 (R/~{W}), U3.24 (P24)
- new net SD_CS: J2.2 (Pin_2), U1.22 (GPIO17)
- new net SD_MISO: J2.5 (Pin_5), U1.21 (GPIO16)
- new net SD_MOSI: J2.3 (Pin_3), U1.25 (GPIO19)
- new net SD_SCK: J2.4 (Pin_4), U1.24 (GPIO18)
- new net STP0: U2.29 (P1)
- new net STP0_3V3: U1.9 (GPIO6)
- new net STP1: U2.30 (P0)
- new net STP1_3V3: U1.10 (GPIO7)
- new net SYNC_3V3: R3.2, U1.4 (GPIO2), U3.56 (P56)
- new net TCK: J5.3 (Pin_3), U3.30 (TCK)
- new net TDI: J5.4 (Pin_4), U3.28 (TDI)
- new net TDO: J5.5 (Pin_5), U3.53 (TDO)
- new net TMS: J5.2 (Pin_2), U3.29 (TMS)
- new net WPS: U2.26 (P4)
- new net WPS_3V3: U1.7 (GPIO5)
- new net XR/~{W}: U3.40 (P40), U7.27 (~{WE})
- new net YB0: U1.11 (GPIO8), U3.22 (P22)
- new net YB1: U1.12 (GPIO9), U3.27 (P27)
- new net YB2: U1.14 (GPIO10), U3.32 (P32)
- new net YB3: U1.15 (GPIO11), U3.33 (P33)
- new net YB4: U1.16 (GPIO12), U3.34 (P34)
- new net YB5: U1.17 (GPIO13), U3.35 (P35)
- new net YB6: U1.19 (GPIO14), U3.36 (P36)
- new net YB7: U1.20 (GPIO15), U3.38 (P38)
- new net ~{CS_TPI}: U3.39 (P39), U5.5 (O1)
- new net ~{E2}: U5.15 (E), U5.6 (O2)
- new net ~{IRQ}: JP3.1 (A), R25.2, U2.3 (~{IRQ})
- new net ~{RAMSEL}: U6.6, U7.20 (~{CS}), U7.22 (~{OE})
- new net ~{RAM_HIGH}: U5.12 (O0), U6.2
- new net ~{RAM_LOW}: U5.4 (O0), U6.1
- new net ~{ROMSEL}: U4.20 (~{CE}), U4.22 (~{OE}), U6.11
- new net ~{ROM_HIGH}: U5.7 (O3), U6.10
- new net ~{ROM_LOW}: U5.11 (O1), U6.9
- no-connect marks 1 -> 14
Other:
- note added: "23x18mm SD Card module 3.3v"
- note added: "ACT_3V3 - converted and inverted ACT"
- note added: "GPIO3 pico"
- note added: "J1: - switch chooses ROM from 32K half of 27C512 closed = bottom half open = top half"
- note added: "NOTE: ACK/DAV naming reversed to keep the TCBM2SD connector intact NOTE: ACK here is controller's ACK output and goes to cable pin 13 (drive's DAV input) NOTE: DAV here is controller's DAV input and goes to cable pin 11 (drive's ACK output) NOTE: DEVNUM_BRD is shorted to GND onboard with hard to use J1 to be cut to pull it up control it on daughterboard NOTE: ~{CS_TPI} is the signal we need to cl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"
- note added: "NOTE: DEVNUM_3V3 - driven by Pico to choose device number, NOT connected to DEVNUM_BRD"
- note added: "NOTE: WPS can be disconnected from board and controled on daughterboard NOTE: DS0/DS1 not connected to pico, no way for unusual formats like SuperDOS? (unless it's not needed at all for G64) NOTE: Phi2 NC onboard, AEC pulled up"
- note added: "NOTE: no macrocells left to use CPLD for level shifting NOTE: all _3V3 signals are for Pico only, NOT for board NOTE: YB0..7 are for Pico only TODO: RESET_3V3, MODE_3V3, SYNC_3V3 NOTE: XR/~{W} comes from GATE ARRAY, it is NOT CPU's R/~{W} CPLD firmware can be later changed to use R/~{W} + Phi0/Phi2 without gate array"
- note added: "Phi0"
- note added: "Pico firmware TODO: - GPIO0: SOE not used (always high), can be fixed in firmware to true - GPIO3: Pico decides about device number - 0 or 1 - GPIO5: switch driver from high/low to hi-z/low - GPIO6,7: STP0/1 just in case (1541 didn't use them) OR - GPIO0: output 2MHz system clock - GPIO3: output 100Hz irq buffer both through 74AHCT1G125"
- note added: "Placeholder only - will do conversion+negation on BSS138 (double check pinout vs footprint!)"
- note added: "TODO: (firmware) - XR/~{W} is OUTPUT, phi2 AND R/W, typical circuit"
- note added: "TODO: - konwersja napiec HIGH->LOW (CAS->TAP - WRITE) MTR, STP0, STP1 - konwersja napiec LOW->HIGH (TAP->CAS - READ), WPS, IRQ - konwersje zrobic jak jak w Pico na mosfet, bo z Pi1551 (CAS->TAP) to inwerter - system clock (z oryginalu) - reset circuit (z oryginalu); RESET 5V vs 3V - dioda albo CPLD, ale nie oba naraz - irq timer (z oryginalu) - albo GPIO0 z PWM do którkich impulsów LOW + level sh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"
- note added: "TODO: falstad sim 100Hz TODO: SMD footprints (also NE555) TODO: JLCPCB partnums"
- note added: "place to tie in GPIO0 (after level shift)"
- note added: "place to tie in divider if more than 2MHz or GPIO3+buffer+R"
- note removed: "(image matches looking at the back of C16/+4)"
- note removed: "B"
- note removed: "C"
- note removed: "E"
- note removed: "JP1 1-2: CAS_SENSE driven by Pi1551 2-3: CAS_SENSE always enabled (resistors and transistor optional)"
- note removed: "JP2 1-2: TAP_MOTOR driven by C16/116/+4 2-3: TAP_MOTOR always enabled (with 6510 CPU replacement) (resistors and transistor optional)"
- note removed: "Note: This must be connected to 5V from tape port, NOT 5V power from RPi!"
- note removed: "TAPE EMULATOR"
- note removed: "all of these TAP_xxx -> CAS_xxx and CAS_xxx -> TAP_xxx converters reverse the logic levels all transistors are NPN: 2n3904 / BC547 / S8050 / etc. Note: SMD transistors have different pinouts THT: B on 2 and E on 1 (EBC) (2N3904) SMD: B on 1 and E on 2 (BEC) (MMBT3904 also sold as 2n3904)"
- title: PI1541-III Module (rotated) -> 1551-III-Pico

Commit message: pico1551-iii schematic revised according to pico1551 discoveries
Parts:
- removed C6: 0.1uF, Capacitor_SMD:C_0805_2012Metric_Pad1.18x1.45mm_HandSolder, symbol Device:C_Small
- removed C7: 10nF, symbol Device:C_Small
- removed C9: 100nF, symbol Device:C_Small
- removed D1: BAT54, Diode_SMD:D_SOD-123, symbol Device:D_Schottky
- removed JP1: ~, Jumper:SolderJumper-2_P1.3mm_Open_RoundedPad1.0x1.5mm, symbol Jumper:SolderJumper_2_Open
- removed JP2, JP3: Jumper_2_Bridged, Connector_PinHeader_2.54mm:PinHeader_1x02_P2.54mm_Vertical, symbol Jumper:Jumper_2_Bridged
- removed Q1: MMBT3904, Package_TO_SOT_SMD:SOT-23_Handsoldering, symbol Transistor_BJT:MMBT3904
- removed R11, R16, R8: 3.3K, Resistor_SMD:R_0805_2012Metric_Pad1.20x1.40mm_HandSolder, symbol Device:R
- removed U8: NE555P, Package_DIP:DIP-8_W7.62mm, symbol Timer:NE555P
- removed U9: 74AHCT1G125, symbol 74xGxx:74AHCT1G125
- removed Y1: 2MHz, Oscillator:Oscillator_DIP-14, symbol Oscillator:CXO_DIP14
- added C11: 10µ, Capacitor_Tantalum_SMD:CP_EIA-3216-12_Kemet-S_HandSolder, symbol Device:C_Polarized
- added JP1, JP2, JP3, JP4: SolderJumper_3_Bridged12, Jumper:SolderJumper-3_P1.3mm_Bridged12_RoundedPad1.0x1.5mm_NumberLabels, symbol Jumper:SolderJumper_3_Bridged12
- added Q1, Q2, Q3, Q4, Q5, Q6: BSS138, Package_TO_SOT_SMD:SOT-23, symbol Transistor_FET:BSS138
- added R1, R19, R27, R28, R29, R30, R31, R32, R33, R34: 3.3K, Resistor_SMD:R_0805_2012Metric_Pad1.20x1.40mm_HandSolder, symbol Device:R
- added R22: 2.2R, Resistor_SMD:R_0805_2012Metric_Pad1.20x1.40mm_HandSolder, symbol Device:R
- added U8: 74HCT165, Package_SO:SOP-16_4.4x10.4mm_P1.27mm, symbol 74xx:74HC165
- added XS1: SD connector, SD2IECplug:Conn_uSDcard, symbol uSD_push-push_ebay:SD_ebay-uSD-push/push_SMD
- J2: renamed from J6; now left out of the parts list
- J3: renamed from J5; now left out of the parts list
- J6: renamed from J2; now left out of the parts list
- R23: value 100 -> 3.3K; JLCPCB Part # (none) -> C26010; JLCPCB URL (none) -> https://jlcpcb.com/partdetail/26753-0805W8F3301T5E/C26010; MFR.Part # (none) -> 0805W8F3301T5E
- R24: value 150K -> 3.3K; JLCPCB Part # (none) -> C26010; JLCPCB URL (none) -> https://jlcpcb.com/partdetail/26753-0805W8F3301T5E/C26010; MFR.Part # (none) -> 0805W8F3301T5E
- R26: value 68 -> 3.3K; JLCPCB Part # (none) -> C26010; JLCPCB URL (none) -> https://jlcpcb.com/partdetail/26753-0805W8F3301T5E/C26010; MFR.Part # (none) -> 0805W8F3301T5E
- SWDBG1, U1, U2: now left out of the parts list
- U4: renamed from U7; now left out of the parts list
- U5: renamed from U4; now left out of the parts list
- U6: renamed from U5; footprint Package_DIP:DIP-16_W7.62mm_Socket_LongPads -> Package_SO:SOP-16_4.4x10.4mm_P1.27mm; JLCPCB Part # (none) -> C521174; JLCPCB URL (none) -> https://www.lcsc.com/product-detail/C521174.html; MFR.Part # (none) -> XL74LS139
- U7: renamed from U6; footprint Package_DIP:DIP-14_W7.62mm_Socket_LongPads -> Package_SO:SO-14_5.3x10.2mm_P1.27mm; JLCPCB Part # (none) -> C609793; JLCPCB URL (none) -> https://www.lcsc.com/product-detail/C609793.html; MFR.Part # (none) -> XL74LS00
- renumbered C13 to C1, C11 to C10, C12 to C2, C2 to C3, C3 to C4, C4 to C5, C5 to C6, C1 to C7, C10 to C9, J3 to J1, J1 to J4, J4 to J5, R17 to R10, R18 to R11, R19 to R12, R20 to R13, R21 to R14, R22 to R15, R1 to R16, R2 to R17, R3 to R18, R4 to R2, R12 to R20, R13 to R21, R5 to R3, R6 to R4, R7 to R5, R9 to R6, R10 to R7, R14 to R8, R15 to R9
Connections:
- net +3V3: now also R23.1, R24.1, R26.1, JP4.3 (B), Q1.1 (G), Q3.1 (G), Q4.1 (G), Q5.1 (G), Q6.1 (G), R19.1, R22.2, R27.1, R29.1, R31.1, R33.1
- net +5V: now also R1.1, R28.1, R30.1, R32.1, R34.1, U8.16 (VCC); no longer R24.1
- net ACT: now also Q2.1 (G)
- net ACT_3V3: now also R26.2, Q2.3 (D)
- net AEC: now also R1.2
- net DEVNUM_3V3: now also JP4.2 (C); no longer U1.5 (GPIO3)
- net DS0: now also U8.14 (D3)
- net DS1: now also U8.3 (D4)
- net GND: now also C11.2, JP4.1 (A), Q2.2 (S), U8.10 (DS), U8.15 (~{CE}), U8.8 (GND), XS1.1 (DAT2), XS1.6 (GND), XS1.8 (DAT1)
- net MTR: now also R25.2, Q1.3 (D)
- net MTR_3V3: now also R24.2, Q1.2 (S)
- net PHI0: now also U1.1 (GPIO0)
- net ROT_CLK: now also JP3.3 (B), U8.12 (D1); no longer U1.31 (GPIO26_ADC0)
- net ROT_DT: now also JP2.3 (B), U8.13 (D2); no longer U1.32 (GPIO27_ADC1)
- net ROT_SW: now also JP1.3 (B), U8.11 (D0); no longer U1.34 (GPIO28_ADC2)
- net SD_CS: now also XS1.2 (CS/DAT3)
- net SD_MISO: now also XS1.7 (DO/DAT0)
- net SD_MOSI: now also XS1.3 (DI/CMD)
- net SD_SCK: now also XS1.5 (CLK)
- net STP0: now also Q3.3 (D), R28.2
- net STP0_3V3: now also Q3.2 (S), R27.2
- net STP1: now also Q5.3 (D), R32.2
- net STP1_3V3: now also Q5.2 (S), R31.2
- net WPS: now also Q6.3 (D), R34.2
- net WPS_3V3: now also Q6.2 (S), R33.2
- net ~{IRQ}: now also U1.5 (GPIO3); no longer R25.2
- net ~{RESET_3V3}: now also R19.2; no longer U3.51 (P51)
- net SD_CD: now reaches R23.2
- net SD_CD: now also U8.4 (D5), XS1.9 (CD)
- new net: C11.1, R22.1, XS1.4 (Vdd)
- new net ROT_CLK_PICO: JP3.2 (C), U1.31 (GPIO26_ADC0)
- new net ROT_DT_PICO: JP2.2 (C), U1.32 (GPIO27_ADC1)
- new net ROT_SW_PICO: JP1.2 (C), U1.34 (GPIO28_ADC2)
- new net SERIAL_CLK: JP2.1 (A), U8.2 (CP)
- new net SERIAL_DT: Q4.3 (D), R30.2, U8.9 (Q7)
- new net SERIAL_DT_3V3: JP1.1 (A), Q4.2 (S), R29.2
- new net SERIAL_LOAD: JP3.1 (A), U8.1 (~{PL})
- no-connect marks 14 -> 18
Other:
- note added: "ACT is active low (LED goes to 5V) ACT_3V3 is active high (LED goes to GND)"
- note added: "ACT_3V3 - converted and inverted ACT (the other side of LED is connected to GND)"
- note added: "Connection block: if shift register idea fails reconnect Pico to encoder"
- note added: "GND - #8 3V3 - #9"
- note added: "NOTE: ACK/DAV naming reversed to keep the TCBM2SD connector intact NOTE: ACK here is controller's ACK output and goes to cable pin 13 (drive's DAV input) NOTE: DAV here is controller's DAV input and goes to cable pin 11 (drive's ACK output) NOTE: ~{CS_TPI} is the signal we need to clear BYTE_LATCHED (aka TED from GATE ARRAY) NOTE: MODE==OE from GATE ARRAY"
- note added: "NOTE: DS0/DS1 connected through shift register NOTE: P3 ACT LED goes between ACT and VCC"
- note added: "Pico firmware: - encoder, DS0/DS1, SD card change from shift register - GPIO0: output 2MHz system clock - GPIO3: output 100Hz irq (buffer both through 74AHCT1G125?)"
- note added: "REVIEW each part: - front panel connector signals - 6502 MOS replacer socket + logic (HCT parts) - all JLCPCB parts, TSSOP"
- note added: "XR/~{W} is OUTPUT: !((!R/~{W} AND PHI2) typical qualified R/W circuit for 6502 peripherals"
- note added: "input GPIO: encoder pins inputs: 3x encoder, 2x DS0/DS1, 1x SD card switch (6 of 8) power: 5V, musi być HCT package: same as cpu replacer thingy CP=clock z pico Q7=data do pico (przez level shift) ~{PL}=load strobe z pico ~{CE}->GND DS->GND (serial input)"
- note removed: "ACT_3V3 - converted and inverted ACT"
- note removed: "GPIO3 pico"
- note removed: "NOTE: ACK/DAV naming reversed to keep the TCBM2SD connector intact NOTE: ACK here is controller's ACK output and goes to cable pin 13 (drive's DAV input) NOTE: DAV here is controller's DAV input and goes to cable pin 11 (drive's ACK output) NOTE: DEVNUM_BRD is shorted to GND onboard with hard to use J1 to be cut to pull it up control it on daughterboard NOTE: ~{CS_TPI} is the signal we need to cl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"
- note removed: "NOTE: DEVNUM_3V3 - driven by Pico to choose device number, NOT connected to DEVNUM_BRD"
- note removed: "NOTE: WPS can be disconnected from board and controled on daughterboard NOTE: DS0/DS1 not connected to pico, no way for unusual formats like SuperDOS? (unless it's not needed at all for G64) NOTE: Phi2 NC onboard, AEC pulled up"
- note removed: "Phi0"
- note removed: "Pico firmware TODO: - GPIO0: SOE not used (always high), can be fixed in firmware to true - GPIO3: Pico decides about device number - 0 or 1 - GPIO5: switch driver from high/low to hi-z/low - GPIO6,7: STP0/1 just in case (1541 didn't use them) OR - GPIO0: output 2MHz system clock - GPIO3: output 100Hz irq buffer both through 74AHCT1G125"
- note removed: "Placeholder only - will do conversion+negation on BSS138 (double check pinout vs footprint!)"
- note removed: "Required b/c depending on tcbm2sd version ~{RESET} can be pulled to 5V or 3.3V use BAT54, BAS40, BAT43, 1n5819 as D2"
- note removed: "TODO: (firmware) - XR/~{W} is OUTPUT, phi2 AND R/W, typical circuit"
- note removed: "TODO: - konwersja napiec HIGH->LOW (CAS->TAP - WRITE) MTR, STP0, STP1 - konwersja napiec LOW->HIGH (TAP->CAS - READ), WPS, IRQ - konwersje zrobic jak jak w Pico na mosfet, bo z Pi1551 (CAS->TAP) to inwerter - system clock (z oryginalu) - reset circuit (z oryginalu); RESET 5V vs 3V - dioda albo CPLD, ale nie oba naraz - irq timer (z oryginalu) - albo GPIO0 z PWM do którkich impulsów LOW + level sh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"
- note removed: "TODO: falstad sim 100Hz TODO: SMD footprints (also NE555) TODO: JLCPCB partnums"
- note removed: "place to tie in GPIO0 (after level shift)"
- note removed: "place to tie in divider if more than 2MHz or GPIO3+buffer+R"
- moved on the sheet: C1, C10, C2, C9, J2, J6, R15, R16, R17, R18, U4, U5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

Commit message: mos6502 replacer integrated
Parts:
- removed R19: 3.3K, Resistor_SMD:R_0805_2012Metric_Pad1.20x1.40mm_HandSolder, symbol Device:R
- added C12, C13, C14, C15, C16, C17: 0.1uF, Capacitor_SMD:C_0805_2012Metric_Pad1.18x1.45mm_HandSolder, symbol Device:C_Small
- added D1, D10, D11, D12, D13, D14, D15, D16, D2, D3, D4, D5, D6, D7, D8, D9: 1N4148W, Diode_SMD:D_SOD-323, symbol Diode:1N4148W
- added JP5: Open for W65C02, Jumper:SolderJumper-2_P1.3mm_Bridged_RoundedPad1.0x1.5mm, symbol Jumper:SolderJumper_2_Bridged
- added R16, R18, R21, R24, R34, R40, R41, R42, R43, R44: 3.3K, Resistor_SMD:R_0805_2012Metric_Pad1.20x1.40mm_HandSolder, symbol Device:R
- added R29: 470, Resistor_SMD:R_0805_2012Metric_Pad1.20x1.40mm_HandSolder, symbol Device:R
- added U1, U10, U2: HCT126, Custom KiCad Library:TSSOP-14_4.4x5mm_P0.65mm, symbol 74xx:74LS126
- added U11: 6502, Package_DIP:DIP-40_W15.24mm_Socket, symbol 6502:6502
- added U13, U14, U16, U18, U7: HCT245, Custom KiCad Library:TSSOP-20_4.4x6.5mm_P0.65mm, symbol 74xx:74LS245
- added U17, U8: HCT273, Custom KiCad Library:TSSOP-20_4.4x6.5mm_P0.65mm, symbol 74xx:74LS273
- added U20: HCT138, Custom KiCad Library:TSSOP-16_4.4x5mm_P0.65mm, symbol 74xx:74LS138
- renumbered C8 to C10, C9 to C8, C10 to C9, R15 to R1, R9 to R10, R10 to R11, R11 to R12, R12 to R13, R13 to R14, R14 to R15, R16 to R17, R17 to R19, R1 to R2, R18 to R20, R20 to R22, R21 to R23, R24 to R25, R25 to R26, R26 to R27, R23 to R28, R2 to R3, R27 to R30, R28 to R31, R29 to R32, R30 to R33, R31 to R35, R32 to R36, R22 to R37, R33 to R38, R34 to R39, R3 to R4, R4 to R5, R5 to R6, R6 to R7, R7 to R8, R8 to R9, U6 to U12, U7 to U15, U8 to U19, U1 to U3, U2 to U6, U3 to U9
Connections:
- net +3.3V: now also R40.2, R41.2, R42.2, R43.2, R44.2
- net +5V: now also C12.1, C13.1, C14.1, C15.1, C16.1, C17.1, R16.1, R18.1, R21.1, R24.2, R29.2, U1.13, U1.14 (VCC), U10.14 (VCC), U11.38 (~{S0}), U11.8 (VCC), U13.1 (A->B), U13.20 (VCC), U14.1 (A->B), U14.20 (VCC), U16.20 (VCC), U17.20 (VCC), U18.1 (A->B), U18.20 (VCC), U2.14 (VCC), U20.16 (VCC), U20.3 (A2), U20.6 (E3), U7.1 (A->B), U7.20 (VCC), U8.20 (VCC)
- net A0: now also U13.11 (B7)
- net A1: now also U13.12 (B6)
- net A10: now also U7.13 (B5)
- net A11: now also U7.14 (B4)
- net A12: now also U7.15 (B3)
- net A13: now also U7.16 (B2)
- net A14: now also U7.17 (B1)
- net A15: now also U7.18 (B0)
- net A2: now also U13.13 (B5)
- net A3: now also U13.14 (B4)
- net A4: now also U13.15 (B3)
- net A5: now also U13.16 (B2)
- net A6: now also U13.17 (B1)
- net A7: now also U13.18 (B0)
- net A8: now also U7.11 (B7)
- net A9: now also U7.12 (B6)
- net ACT: now also U14.5 (A3), U2.11
- net AEC: now also D16.2 (A), R29.1, U1.6, U1.9, U13.19 (CE), U7.19 (CE); no longer R2.2, U6.4 (AEC)
- net BYTE_LATCHED: now also U10.11, U14.9 (A7)
- net D0: now also U16.9 (A7)
- net D1: now also U16.8 (A6)
- net D2: now also U16.7 (A5)
- net D3: now also U16.6 (A4)
- net D4: now also U16.5 (A3)
- net D5: now also U16.4 (A2)
- net D6: now also U16.3 (A1)
- net D7: now also U16.2 (A0)
- net DS0: now also U10.6, U14.7 (A5)
- net DS1: now also U10.8, U14.8 (A6)
- net GND: now also C12.2, C13.2, C14.2, C15.2, C16.2, C17.2, JP5.1 (A), R34.1, U1.5, U1.7 (GND), U10.7 (GND), U11.21 (GND), U13.10 (GND), U14.10 (GND), U16.10 (GND), U17.10 (GND), U18.10 (GND), U2.7 (GND), U20.5 (E2), U20.8 (GND), U7.10 (GND), U8.10 (GND)
- net MTR: now also U14.4 (A2), U2.8
- net PHI0: now also U11.37 (PHI0IN)
- net PHI2: now also U1.11
- net ROT_CLK: now also R43.1
- net ROT_DT: now also R42.1
- net ROT_SW: now also R44.1
- net R/~{W}: now also U1.3
- net SW4_BACK: now also U19.5 (D6), R40.1
- net SW5_INSERT: now also U19.6 (D7), R41.1
- net ~{IRQ}: now also U11.4 (~{IRQ})
- net ~{RESET}: now also U11.40 (~{RESET}), U17.1 (~{Mr}), U8.1 (~{Mr})
- net STP0 renamed P1
- net P1: now also U14.3 (A1), U2.6
- net STP1 renamed P0
- net P0: now also U14.2 (A0), U2.3
- net WPS renamed P4
- net P4: now also U10.3, U14.6 (A4)
- new net: R24.1, U1.8, U16.19 (CE)
- new net: JP5.2 (B), U11.1 (GND)
- new net: R21.2, U11.36 (NC)
- new net: U1.12, U11.39 (PHI2OUT)
- new net CA0: U11.9 (A0), U13.9 (A7), U20.1 (A0)
- new net CA1: D1.2 (A), U11.10 (A1), U13.8 (A6)
- new net CA10: D10.2 (A), U11.19 (A10), U7.7 (A5)
- new net CA11: D11.2 (A), U11.20 (A11), U7.6 (A4)
- new net CA12: D12.2 (A), U11.22 (A12), U7.5 (A3)
- new net CA13: D13.2 (A), U11.23 (A13), U7.4 (A2)
- new net CA14: D14.2 (A), U11.24 (A14), U7.3 (A1)
- new net CA15: D15.2 (A), U11.25 (A15), U7.2 (A0)
- new net CA2: D2.2 (A), U11.11 (A2), U13.7 (A5)
- new net CA3: D3.2 (A), U11.12 (A3), U13.6 (A4)
- new net CA4: D4.2 (A), U11.13 (A4), U13.5 (A3)
- new net CA5: D5.2 (A), U11.14 (A5), U13.4 (A2)
- new net CA6: D6.2 (A), U11.15 (A6), U13.3 (A1)
- new net CA7: D7.2 (A), U11.16 (A7), U13.2 (A0)
- new net CA8: D8.2 (A), U11.17 (A8), U7.9 (A7)
- new net CA9: D9.2 (A), U11.18 (A9), U7.8 (A6)
- new net CD0: U11.33 (D0), U14.18 (B0), U16.11 (B7), U17.3 (D0), U18.18 (B0), U8.3 (D0)
- new net CD1: U11.32 (D1), U14.17 (B1), U16.12 (B6), U17.4 (D1), U18.17 (B1), U8.4 (D1)
- new net CD2: U11.31 (D2), U14.16 (B2), U16.13 (B5), U17.7 (D2), U18.16 (B2), U8.7 (D2)
- new net CD3: U11.30 (D3), U14.15 (B3), U16.14 (B4), U17.8 (D3), U18.15 (B3), U8.8 (D3)
- new net CD4: U11.29 (D4), U14.14 (B4), U16.15 (B3), U17.13 (D4), U18.14 (B4), U8.13 (D4)
- new net CD5: U11.28 (D5), U14.13 (B5), U16.16 (B2), U17.14 (D5), U18.13 (B5), U8.14 (D5)
- new net CD6: U11.27 (D6), U14.12 (B6), U16.17 (B1), U17.17 (D6), U18.12 (B6), U8.17 (D6)
- new net CD7: U11.26 (D7), U14.11 (B7), U16.18 (B0), U17.18 (D7), U18.11 (B7), U8.18 (D7)
- new net DAT0: U2.2, U8.2 (Q0)
- new net DAT1: U2.5, U8.5 (Q1)
- new net DAT2: U2.9, U8.6 (Q2)
- new net DAT3: U2.12, U8.9 (Q3)
- new net DAT4: U10.2, U8.12 (Q4)
- new net DAT5: U10.5, U8.15 (Q5)
- new net DAT6: U10.9, U8.16 (Q6)
- new net DAT7: U10.12, U8.19 (Q7)
- new net DIR0: U17.2 (Q0), U18.2 (A0), U2.1
- new net DIR1: U17.5 (Q1), U18.3 (A1), U2.4
- new net DIR2: U17.6 (Q2), U18.4 (A2), U2.10
- new net DIR3: U17.9 (Q3), U18.5 (A3), U2.13
- new net DIR4: U10.1, U17.12 (Q4), U18.6 (A4)
- new net DIR5: U10.4, U17.15 (Q5), U18.7 (A5)
- new net DIR6: U10.10, U17.16 (Q6), U18.8 (A6)
- new net DIR7: U10.13, U17.19 (Q7), U18.9 (A7)
- new net RDY: R18.2, U11.2 (RDY)
- new net ~{0000-0001}: D1.1 (K), D10.1 (K), D11.1 (K), D12.1 (K), D13.1 (K), D14.1 (K), D15.1 (K), D16.1 (K), D2.1 (K), D3.1 (K), D4.1 (K), D5.1 (K), D6.1 (K), D7.1 (K), D8.1 (K), D9.1 (K), R34.2, U1.10, U20.4 (E1)
- new net ~{0000_RD}: U18.19 (CE), U20.9 (O6)
- new net ~{0000_WR}: U17.11 (Cp), U20.11 (O4)
- new net ~{0001_RD}: U14.19 (CE), U20.7 (O7)
- new net ~{0001_WR}: U20.10 (O5), U8.11 (Cp)
- new net ~{6502RW}: U1.2, U11.34 (R/~{W}), U16.1 (A->B), U20.2 (A1)
- new net ~{AEC}: R2.2, U1.1, U1.4, U6.4 (AEC)
- new net ~{NMI}: R16.2, U11.6 (~{NMI})
- no-connect marks 18 -> 24
Other:
- note added: "Clock buffer added in Rev2. Should fix C64 compatibility issues, and maybe some others. Thanks to Ray of Retro Tech Insanity."
- note added: "For *65C02 support"
- note added: "Only open JP1 for WDC W65C02, not other 65C02. Using a *65C02 will result in reduced software compatibility due to CPU bugs fixed and undocumented opcodes altered, which are exploited by some software/games/demos."
- note added: "Pico firmware: - encoder, DS0/DS1, SD card change from shift register, SW4, SW5 - GPIO0: output 2MHz system clock - GPIO3: output 100Hz irq (buffer both through 74AHCT1G125?) - footprints - SW4/SW5 need pullups?"
- note added: "REVIEW each part: - front panel connector signals - 6502 MOS replacer socket + logic (HCT parts) - all JLCPCB parts, TSSOP - additional footprints: Pico, SD card"
- note removed: "Pico firmware: - encoder, DS0/DS1, SD card change from shift register - GPIO0: output 2MHz system clock - GPIO3: output 100Hz irq (buffer both through 74AHCT1G125?)"
- note removed: "REVIEW each part: - front panel connector signals - 6502 MOS replacer socket + logic (HCT parts) - all JLCPCB parts, TSSOP"

Commit message: all the footprints from other projects
Parts:
- SYM1: footprint BulkyMIDI-32:PWR_Specification -> pi1541:PWR_Specification
Changed lines of the file:
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@@
 			)
 		)
-		(property "Footprint" "BulkyMIDI-32:PWR_Specification"
+		(property "Footprint" "pi1541:PWR_Specification"
 			(at 58.42 167.005 0)
 			(effects

Commit message: part placement and routing test
Parts:
- removed C12, C13, C14, C15, C16, C17: 0.1uF, Capacitor_SMD:C_0805_2012Metric_Pad1.18x1.45mm_HandSolder, symbol Device:C_Small
- removed D1, D10, D11, D12, D13, D14, D15, D16, D2, D3, D4, D5, D6, D7, D8, D9: 1N4148W, Diode_SMD:D_SOD-323, symbol Diode:1N4148W
- removed JP4: SolderJumper_3_Bridged12, Jumper:SolderJumper-3_P1.3mm_Bridged12_RoundedPad1.0x1.5mm_NumberLabels, symbol Jumper:SolderJumper_3_Bridged12
- removed JP5: Open for W65C02, Jumper:SolderJumper-2_P1.3mm_Bridged_RoundedPad1.0x1.5mm, symbol Jumper:SolderJumper_2_Bridged
- removed R21, R24, R34: 3.3K, Resistor_SMD:R_0805_2012Metric_Pad1.20x1.40mm_HandSolder, symbol Device:R
- removed R29: 470, Resistor_SMD:R_0805_2012Metric_Pad1.20x1.40mm_HandSolder, symbol Device:R
- removed SWDBG1: DEBUG, Connector_PinHeader_2.54mm:PinHeader_1x03_P2.54mm_Vertical, symbol Connector_Generic:Conn_01x03
- removed U1, U10, U2: HCT126, Custom KiCad Library:TSSOP-14_4.4x5mm_P0.65mm, symbol 74xx:74LS126
- removed U11: 6502, Package_DIP:DIP-40_W15.24mm_Socket, symbol 6502:6502
- removed U13, U14, U16, U18, U7: HCT245, Custom KiCad Library:TSSOP-20_4.4x6.5mm_P0.65mm, symbol 74xx:74LS245
- removed U17, U8: HCT273, Custom KiCad Library:TSSOP-20_4.4x6.5mm_P0.65mm, symbol 74xx:74LS273
- removed U20: HCT138, Custom KiCad Library:TSSOP-16_4.4x5mm_P0.65mm, symbol 74xx:74LS138
- added J7: Conn_01x02_Pin, Connector_PinHeader_2.54mm:PinHeader_1x02_P2.54mm_Vertical, symbol Connector:Conn_01x02_Pin
Connections:
- net RDY is gone; now on net DEVNUM_3V3: R18.2
- net ~{NMI} is gone; now on net ~{RESET}: R16.2
- net +3V3: now also R18.1
- net +5V: no longer R18.1
- net DEVNUM_3V3: now also J7.1 (Pin_1)
- net GND: now also U3.42 (GND), J7.2 (Pin_2)
- net P0 renamed STP1
- net P1 renamed STP0
- net P4 renamed WPS
- no-connect marks 24 -> 18
Other:
- note added: "GND - #8 - closed 3V3 - #9 - open"
- note added: "REVIEW each part: - front panel connector signals - all JLCPCB parts, TSSOP"
- note removed: "Clock buffer added in Rev2. Should fix C64 compatibility issues, and maybe some others. Thanks to Ray of Retro Tech Insanity."
- note removed: "For *65C02 support"
- note removed: "GND - #8 3V3 - #9"
- note removed: "Only open JP1 for WDC W65C02, not other 65C02. Using a *65C02 will result in reduced software compatibility due to CPU bugs fixed and undocumented opcodes altered, which are exploited by some software/games/demos."
- note removed: "REVIEW each part: - front panel connector signals - 6502 MOS replacer socket + logic (HCT parts) - all JLCPCB parts, TSSOP - additional footprints: Pico, SD card"

Commit message: project updated and routed: IRQ with pullup, correct 3V3 net, correct inputs for '139
Parts:
- added R21: 3.3K, Resistor_SMD:R_0805_2012Metric_Pad1.20x1.40mm_HandSolder, symbol Device:R
Connections:
- net +3.3V is gone; now on net +3V3: J5.12 (VCC), R10.1, R11.1, R12.1, R13.1, R14.1, R15.1, R22.2, R3.1, R4.1, R40.2, R41.2, R42.2, R43.2, R44.2, R5.1, R6.1, R7.1, R8.1, R9.1
- net +3V3: now also R21.1
- net A13: now also U12.14 (A0); no longer U12.13 (A1)
- net A14: now also U12.2 (A0); no longer U12.3 (A1)
- net A15: now also U12.3 (A1); no longer U12.2 (A0)
- net GND: now also U12.13 (A1); no longer U12.14 (A0)
- net ~{IRQ}: now also R21.2
Other:
- note added: "Pico firmware: - encoder, DS0/DS1, SD card change from shift register, SW4, SW5 - GPIO0: output 2MHz system clock - GPIO3: output 100Hz irq"
- note removed: "Pico firmware: - encoder, DS0/DS1, SD card change from shift register, SW4, SW5 - GPIO0: output 2MHz system clock - GPIO3: output 100Hz irq (buffer both through 74AHCT1G125?) - footprints - SW4/SW5 need pullups?"
