File: hardware-1551-III-Pico/1551-III-Pico.kicad_sch (KiCad schematic)
At the start: 82 parts, among them J1 TCBM, J2 Conn_01x02_Pin, J3 JTAG, J4 DC IN, J5 Module_Panel, J6 SD CARD, J7 Conn_01x02_Pin, M1 Mounting, M2 Mounting, M3 Mounting, M4 Mounting, Q1 BSS138, Q2 BSS138, Q3 BSS138, Q4 BSS138, Q5 BSS138, Q6 BSS138, U12 74LS139, U15 74LS00, U19 74HCT165, U3 Pico, U4 KM62256CLP, U5 27C512, U6 6510T, U9 XC9572XL-VQ64

Commit message: remove '139 and '00 logic to embed it into CPLD, routed final version
Parts:
- removed C8, C9: 0.1uF, Capacitor_SMD:C_0805_2012Metric_Pad1.18x1.45mm_HandSolder, symbol Device:C_Small
- removed U12: 74LS139, Package_SO:SOP-16_4.4x10.4mm_P1.27mm, symbol 74xx:74LS139
- removed U15: 74LS00, Package_SO:SO-14_5.3x10.2mm_P1.27mm, symbol 74xx:74LS00
Connections:
- net ~{CS_TPI} is gone; now on net A14: U9.39 (P39)
- net A13: now also U9.61 (P61)
- net A15: now also U9.62 (P62)
- net ~{RAMSEL}: now also U9.58 (P58); no longer U4.22 (~{OE})
- net ~{ROMSEL}: now also U9.59 (P59)
- net ~{RAMOE}: now reaches U9.42 (P42)
- net ~{RAMOE}: now also U4.22 (~{OE})
- no-connect marks 18 -> 11
Other:
- note added: "NOTE: ACK/DAV naming reversed to keep the TCBM2SD connector intact NOTE: ACK here is controller's ACK output and goes to cable pin 13 (drive's DAV input) NOTE: DAV here is controller's DAV input and goes to cable pin 11 (drive's ACK output) NOTE: MODE==OE from GATE ARRAY"
- note removed: "NOTE: ACK/DAV naming reversed to keep the TCBM2SD connector intact NOTE: ACK here is controller's ACK output and goes to cable pin 13 (drive's DAV input) NOTE: DAV here is controller's DAV input and goes to cable pin 11 (drive's ACK output) NOTE: ~{CS_TPI} is the signal we need to clear BYTE_LATCHED (aka TED from GATE ARRAY) NOTE: MODE==OE from GATE ARRAY"
- note removed: "NOTE: no macrocells left to use CPLD for level shifting NOTE: all _3V3 signals are for Pico only, NOT for board NOTE: YB0..7 are for Pico only TODO: RESET_3V3, MODE_3V3, SYNC_3V3 NOTE: XR/~{W} comes from GATE ARRAY, it is NOT CPU's R/~{W} CPLD firmware can be later changed to use R/~{W} + Phi0/Phi2 without gate array"

Commit message: finalized revision and files for manufacturing
Parts:
- U19: value 74HCT165 -> 74LS165; JLCPCB Part # C42403065 -> C7742; JLCPCB URL https://www.lcsc.com/product-detail/C42403065.html -> https://www.lcsc.com/product-detail/C7742.html; MFR.Part # SN74LS165ADR(LX) -> SN74LS165ADR
Other:
- note removed: "REVIEW each part: - front panel connector signals - all JLCPCB parts, TSSOP"
- note removed: "input GPIO: encoder pins inputs: 3x encoder, 2x DS0/DS1, 1x SD card switch (6 of 8) power: 5V, musi być HCT package: same as cpu replacer thingy CP=clock z pico Q7=data do pico (przez level shift) ~{PL}=load strobe z pico ~{CE}->GND DS->GND (serial input)"
Changed lines of the file:
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@@
 	(title_block
 		(title "1551-III-Pico")
-		(date "2026-08-01")
+		(date "2026-08-16")
 		(rev "2")
 	)
@@
 		)
 	)
-	(text "input GPIO: encoder pins\ninputs: 3x encoder, 2x DS0/DS1, 1x SD card switch (6 of 8)\npower: 5V, musi być HCT\npackage: same as cpu replacer thingy\n\nCP=clock z pico\nQ7=data do pico (przez level shift)\n~{PL}=load strobe z pico\n~{CE}->GND\nDS->GND (serial input)"
-		(exclude_from_sim no)
-		(at 230.759 272.542 0)
-		(effects
-			(font
-				(size 1.27 1.27)
-			)
-			(justify left)
-		)
-	)
 	(text "J1:\n- switch chooses ROM\n  from 32K half of 27C512\n  closed = bottom half\n  open = top half\n"
 		(exclude_from_sim no)
@@
 		)
 	)
-	(text "REVIEW each part:\n- front panel connector signals\n- all JLCPCB parts, TSSOP"
-		(exclude_from_sim no)
-		(at 9.906 -45.72 0)
-		(effects
-			(font
-				(size 3.81 3.81)
-			)
-			(justify left)
-		)
-	)
 	(text "ACT_3V3 - converted and inverted ACT\n(the other side of LED is connected to GND)"
 		(exclude_from_sim no)
@@
 			)
 		)
-		(property "Value" "74HCT165"
+		(property "Value" "74LS165"
 			(at 223.7583 251.46 0)
 			(effects
@@
 			)
 		)
-		(property "Datasheet" "https://assets.nexperia.com/documents/data-sheet/74HC_HCT165.pdf"
+		(property "Datasheet" "https://www.lcsc.com/datasheet/C7742.pdf"
 			(at 221.615 271.78 0)
 			(effects
@@
 			)
 		)
-		(property "JLCPCB Part #" "C42403065"
+		(property "JLCPCB Part #" "C7742"
 			(at 221.615 271.78 0)
 			(effects
@@
 			)
 		)
-		(property "JLCPCB URL" "https://www.lcsc.com/product-detail/C42403065.html"
+		(property "JLCPCB URL" "https://www.lcsc.com/product-detail/C7742.html"
 			(at 221.615 271.78 0)
 			(effects
@@
 			)
 		)
-		(property "MFR.Part #" "SN74LS165ADR(LX)"
+		(property "MFR.Part #" "SN74LS165ADR"
 			(at 221.615 271.78 0)
 			(effects
