File: hardware-1551-III-Pico/1551-III-Pico.kicad_sch (KiCad schematic)
At the start: 78 parts, among them J1 TCBM, J2 Conn_01x02_Pin, J3 JTAG, J4 DC IN, J5 Module_Panel, J6 SD CARD, J7 Conn_01x02_Pin, M1 Mounting, M2 Mounting, M3 Mounting, M4 Mounting, Q1 BSS138, Q2 BSS138, Q3 BSS138, Q4 BSS138, Q5 BSS138, Q6 BSS138, U19 74LS165, U3 Pico, U4 KM62256CLP, U5 27C512, U6 6510T, U9 XC9572XL-VQ64

Commit message: ACT LED corrections after tests: move LED current limiter (R23, 470R) to R27 position (former 3K3 pullup)
Parts:
- removed R23: 470*, Resistor_SMD:R_0805_2012Metric_Pad1.20x1.40mm_HandSolder, symbol Device:R
- R27: value 3.3K -> 470*; JLCPCB Part # C26010 -> C17710; JLCPCB URL https://jlcpcb.com/partdetail/26753-0805W8F3301T5E/C26010 -> https://jlcpcb.com/partdetail/18398-0805W8F4700T5E/C17710; MFR.Part # 0805W8F3301T5E -> 0805W8F4700T5E
Connections:
- net LED_ACT is gone; now on net ACT_3V3: J5.3 (LED_ACT)
Other:
- note added: "Connection block: if shift register idea fails reconnect Pico to encoder (shift register works fine, so this could be removed)"
- note removed: "Connection block: if shift register idea fails reconnect Pico to encoder"
- moved on the sheet: Q2, R27
