File: hardware-1551-III-Pico/1551-III-Pico.kicad_pcb (KiCad board)
At the start: 2 copper layers, 100 x 100 mm, 81 parts, among them J1 TCBM, J2 Conn_01x02_Pin, J3 JTAG, J4 DC IN, J5 Module_Panel, J6 SD CARD, J7 Conn_01x02_Pin, M1 Mounting, M2 Mounting, M3 Mounting, M4 Mounting, Q1 BSS138, Q2 BSS138, Q3 BSS138, Q4 BSS138, Q5 BSS138, Q6 BSS138, U19 74HCT165, U3 Pico, U4 KM62256CLP, U5 27C512, U6 6510T, U9 XC9572XL-VQ64

Commit message: ACT LED corrections after tests: move LED current limiter (R23, 470R) to R27 position (former 3K3 pullup)
Parts:
- removed R23: 470*, Resistor_SMD:R_0805_2012Metric_Pad1.20x1.40mm_HandSolder
- R27: value 3.3K -> 470*
- U19: value 74HCT165 -> 74LS165
Connections:
- J5 pad 3: LED_ACT -> /ACT_3V3
Routing:
- net /ACT_3V3: track 9.65 -> 16.3 mm
- net LED_ACT: track 5.23 -> 0.00 mm
Other:
- board text added: "1551-III-Pico v1.1 Maciej Wiktowiak <ytm@elysium.pl> IX 2026"
- board text added: "O:#9 C:#8"
- board text removed: "1551-III-Pico v1.0 Maciej Wiktowiak <ytm@elysium.pl> VIII 2026"
- board text removed: "C:#9 O:#8"
